Commit message: [Revise] 1.Add color to the Robot model 2. Delete unused world file 3.Solved the Robot Model Spawn Error.

File: project2/my_robot/urdf/my_robot.xacro (robot description, xacro)
@@ -69,7 +69,4 @@
        <cylinder radius ="0.1" length="0.05"/>
      </geometry>
-     <material name="Cyan">
-     <color rgba="0 255 1.0 1.0"/>
-     </material>
    </visual>
    <collision>
@@ -93,7 +90,7 @@
        <cylinder radius ="0.1" length="0.05"/>
      </geometry>
-     <material name="Cyan">
-     <color rgba="0 255 1.0 1.0"/>
-     </material>
+    <material name="red">
+        <color rgba="255 0.1 0.1 1"/>
+      </material>
    </visual>
    <collision>
@@ -116,7 +113,4 @@
        <box size=".05 .05 .05"/>
      </geometry>
-     <material name="Cyan">
-     <color rgba="0 1.0 1.0 1.0"/>
-     </material>
    </visual>
    <collision>
@@ -176,3 +170,7 @@
     <axis xyz="0 1 0" rpy="0 0 0"/>
   </joint>
+ <gazebo reference="chassis"> <material>Gazebo/Yellow</material> </gazebo>
+ <gazebo reference="rightWheel"> <material>Gazebo/Green</material> </gazebo>
+ <gazebo reference="leftWheel"> <material>Gazebo/Green</material> </gazebo>
+ <gazebo reference="camera"> <material>Gazebo/Red</material> </gazebo>
 </robot>
